File: Receiver/IQ_SDR/IQ_SDR.sch (KiCad schematic (older format))
At the start: 83 parts, among them CON1 SJ1-3523N, J1 FIL_I, J10 GNDA, J11 I_IN, J12 Q_IN, J13 I_OUT, J14 Q_OUT, J2 GND, J3 GND, J4 FIL_O, J5 CLK1, J6 CLK2, J7 CLK0, J8 LO_I, J9 LO_Q, P1 BNC, P2 SMA, T1 Transformer_1P_SS, U1 FST3253, U2 Si5351A-B-GT, U3 TS5A23157, U4 SA5532 or LT6231, U5 74ALVC74D, Y1 CX3225

Commit message: More cleanup of schematic
Parts:
- C14, C4: value 1470pF -> 1.47nF
Changed lines of the file:
@@
 EESchema Schematic File Version 4
 LIBS:IQ_SDR-cache
-EELAYER 26 0
+EELAYER 29 0
 EELAYER END
 $Descr USLetter 11000 8500
@@
 U 1 1 5D17E138
 P 2700 3400
-F 0 "L8" V 2890 3400 50  0000 C CNN
+F 0 "L8" V 2650 3400 50  0000 C CNN
 F 1 "7.2uH" V 2799 3400 50  0000 C CNN
 F 2 "Inductors_THT:L_Toroid_Vertical_L10.0mm_W5.0mm_P5.08mm" H 2700 3400 50  0001 C CNN
@@
 U 1 1 5D17E962
 P 2700 3600
-F 0 "C10" V 2448 3600 50  0000 C CNN
-F 1 "486pF" V 2539 3600 50  0000 C CNN
+F 0 "C10" V 2800 3750 50  0000 C CNN
+F 1 "486pF" V 2750 3400 50  0000 C CNN
 F 2 "Capacitors_SMD:C_0805" H 2738 3450 50  0001 C CNN
 F 3 "~" H 2700 3600 50  0001 C CNN
@@
 P 1800 3750
 F 0 "C4" H 1850 3850 50  0000 L CNN
-F 1 "1470pF" H 1700 3950 50  0000 L CNN
+F 1 "1.47nF" H 1550 3950 50  0000 L CNN
 F 2 "Capacitors_SMD:C_0805" H 1838 3600 50  0001 C CNN
 F 3 "~" H 1800 3750 50  0001 C CNN
@@
 U 1 1 5D17EF81
 P 3400 3750
-F 0 "C14" H 3450 3850 50  0000 L CNN
-F 1 "1470pF" H 3100 3650 50  0000 L CNN
+F 0 "C14" H 3200 3850 50  0000 L CNN
+F 1 "1.47nF" H 3100 3650 50  0000 L CNN
 F 2 "Capacitors_SMD:C_0805" H 3438 3600 50  0001 C CNN
 F 3 "~" H 3400 3750 50  0001 C CNN
@@
 U 1 1 5D1D3FF4
 P 2650 3950
-F 0 "L7" V 2840 3950 50  0000 C CNN
+F 0 "L7" V 2600 3950 50  0000 C CNN
 F 1 "4uH" V 2749 3950 50  0000 C CNN
 F 2 "Inductors_THT:L_Toroid_Vertical_L10.0mm_W5.0mm_P5.08mm" H 2650 3950 50  0001 C CNN
@@
 U 1 1 5D1D3FFB
 P 2650 4150
-F 0 "C9" V 2398 4150 50  0000 C CNN
-F 1 "199pF" V 2489 4150 50  0000 C CNN
+F 0 "C9" V 2750 4250 50  0000 C CNN
+F 1 "199pF" V 2700 3950 50  0000 C CNN
 F 2 "Capacitors_SMD:C_0805" H 2688 4000 50  0001 C CNN
 F 3 "~" H 2650 4150 50  0001 C CNN
@@
 U 1 1 5D1D4010
 P 3350 4300
-F 0 "C13" H 3400 4400 50  0000 L CNN
-F 1 "796pF" H 3050 4200 50  0000 L CNN
+F 0 "C13" H 3150 4400 50  0000 L CNN
+F 1 "796pF" H 3100 4200 50  0000 L CNN
 F 2 "Capacitors_SMD:C_0805" H 3388 4150 50  0001 C CNN
 F 3 "~" H 3350 4300 50  0001 C CNN
@@
 U 1 1 5D22E323
 P 2600 4700
-F 0 "C8" V 2348 4700 50  0000 C CNN
+F 0 "C8" V 2700 4800 50  0000 C CNN
 F 1 "100pF" V 2439 4700 50  0000 C CNN
 F 2 "Capacitors_SMD:C_0805" H 2638 4550 50  0001 C CNN
@@
 P 1900 4850
 F 0 "C6" H 1950 4950 50  0000 L CNN
-F 1 "398pF" H 1800 5050 50  0000 L CNN
+F 1 "398pF" H 1650 4950 50  0000 L CNN
 F 2 "Capacitors_SMD:C_0805" H 1938 4700 50  0001 C CNN
 F 3 "~" H 1900 4850 50  0001 C CNN
@@
 U 1 1 5D22E338
 P 3300 4850
-F 0 "C12" H 3350 4950 50  0000 L CNN
-F 1 "398pF" H 3000 4750 50  0000 L CNN
+F 0 "C12" H 3100 4950 50  0000 L CNN
+F 1 "398pF" H 3050 4750 50  0000 L CNN
 F 2 "Capacitors_SMD:C_0805" H 3338 4700 50  0001 C CNN
 F 3 "~" H 3300 4850 50  0001 C CNN
@@
 U 1 1 5D258FC6
 P 2550 5050
-F 0 "L5" V 2740 5050 50  0000 C CNN
+F 0 "L5" V 2500 5050 50  0000 C CNN
 F 1 "1.137uH" V 2649 5050 50  0000 C CNN
 F 2 "Inductors_THT:L_Toroid_Vertical_L10.0mm_W5.0mm_P5.08mm" H 2550 5050 50  0001 C CNN
@@
 U 1 1 5D258FCD
 P 2550 5250
-F 0 "C7" V 2298 5250 50  0000 C CNN
-F 1 "46pF" V 2389 5250 50  0000 C CNN
+F 0 "C7" V 2650 5350 50  0000 C CNN
+F 1 "46pF" V 2650 5100 50  0000 C CNN
 F 2 "Capacitors_SMD:C_0805" H 2588 5100 50  0001 C CNN
 F 3 "~" H 2550 5250 50  0001 C CNN
@@
 P 1800 5400
 F 0 "C5" H 1850 5500 50  0000 L CNN
-F 1 "227pF" H 1700 5600 50  0000 L CNN
+F 1 "227pF" H 1550 5500 50  0000 L CNN
 F 2 "Capacitors_SMD:C_0805" H 1838 5250 50  0001 C CNN
 F 3 "~" H 1800 5400 50  0001 C CNN
@@
 U 1 1 5D258FE2
 P 3250 5400
-F 0 "C11" H 3300 5500 50  0000 L CNN
-F 1 "227pF" H 2950 5300 50  0000 L CNN
+F 0 "C11" H 3050 5500 50  0000 L CNN
+F 1 "227pF" H 3000 5300 50  0000 L CNN
 F 2 "Capacitors_SMD:C_0805" H 3288 5250 50  0001 C CNN
 F 3 "~" H 3250 5400 50  0001 C CNN

Commit message: Changes to power and perhaps a better op amp...
Parts:
- added C24: 10uF, Capacitors_SMD:C_0805, symbol Device:C
- added C28: 0.1uF, Capacitors_SMD:C_0805, symbol Device:C
- added J15: +5V, Connectors:PINTST, symbol Connector_Generic:Conn_01x01
- added J16: 4.3V, Connectors:PINTST, symbol Connector_Generic:Conn_01x01
- added J3: V_IN pin header, symbol Connector_Generic:Conn_01x02
- added J5: Barrel Connector, symbol Connector_Generic:Conn_01x02
- added JP1: Jumper_3_Bridged12, symbol Jumper:Jumper_3_Bridged12
- added Q1: MMBT2222A-TP, digikey-footprints:SOT-23-3, symbol dk_Transistors-Bipolar-BJT-Single:MMBT2222A-TP
- added R8: 1k, Resistors_SMD:R_0805, symbol Device:R
- C10: value 486pF -> 480pF
- C11, C5: value 227pF -> 220pF
- C12, C6: value 398pF -> 390pF
- C13, C2: value 796pF -> 820pF
- C14, C4: value 1.47nF -> 1.5nF
- C31: renamed from C30; value 0.1uF -> 10uF
- C7: value 46pF -> 47pF
- C9: value 199pF -> 200pF
- J1: value FIL_I -> ANT
- U4: value SA5532 or LT6231 -> LM4562 or LT6231
- renumbered C24 to C25, C25 to C26, C26 to C27, C28 to C29, C29 to C30, C27 to C32, J8 to J10, J9 to J11, J10 to J12, J11 to J13, J12 to J14, J13 to J17, J14 to J18, J3 to J4, J4 to J6, J5 to J7, J6 to J8, J7 to J9, R9 to R10, R10 to R11, R11 to R12, R12 to R13, R13 to R14, R8 to R9
Connections:
- net +5V: now also J15.1 (Pin_1), Q1.3 (C), R8.1; no longer C1.1, C16.1, C18.1, C19.1, R2.2, R4.2, R6.1, U1.16 (V+), U3.8 (V+), U4.8 (V+)
- net GND: now also C24.2, C28.2, J3.2 (Pin_2), J5.2 (Pin_2)
- new net: C24.1, Q1.1 (B), R8.2
- new net +4.3V: C1.1, C16.1, C18.1, C28.1, J16.1 (Pin_1), JP1.1 (A), Q1.2 (E), R2.2, R4.2, U1.16 (V+), U3.8 (V+)
- new net V_CC: C19.1, JP1.2 (C), R6.1, U4.8 (V+)
- new net V_IN: J3.1 (Pin_1), J5.1 (Pin_1), JP1.3 (B)
Other:
- note added: "Connect J15\nto J16 to \nremove\neffect of CC\nsmoother."
- note added: "Emitter follower\nto smooth USB\n+5V."
- note added: "External DC in\nto run op amps\nif desired."
- note added: "Inputs for external\nDC input for op\namps."
- note added: "LT6231 has lower noise figure (4.7 dB), \nbut costs about 7 times as much\nas the SA5532. LME49860 is \nintermediate option. LM4562\ncould be even better (10.6 dB)\n2.7nV/sqrt(Hz)."
- note added: "Making T1 a step up\ntransformer makes\nthe S/N and NF better."
- note added: "R9-10 can be\nup to 100\nwith LM4562."
- note added: "V_IN is an optional\nDC Voltage for up to\n+30V."
- note removed: "LT6231 has lower noise figure (6 dB), \nbut costs about 7 times as much\nas the SA5532."
- moved on the sheet: C31, C32

Commit message: Added PCB.
Parts:
- removed J5: Barrel Connector, symbol Connector_Generic:Conn_01x02
- added J19, J20: Conn_01x01_Male, Pin_Headers:Pin_Header_Straight_1x01_Pitch2.54mm, symbol Connector:Conn_01x01_Male
- added J5: V_IN, Connectors:BARREL_JACK, symbol Connector:Barrel_Jack_Switch
- added JP1: smooth disable, Pin_Headers:Pin_Header_Straight_1x02_Pitch2.54mm, symbol Jumper:Jumper_2_Open
- added R15, R16: 4.7k, Resistors_SMD:R_0805, symbol Device:R
- A1: footprint Module:Arduino_Nano -> Modules:Arduino_Nano
- J3: footprint (none) -> Pin_Headers:Pin_Header_Straight_1x02_Pitch2.54mm
- JP2: renamed from JP1; footprint (none) -> Pin_Headers:Pin_Header_Straight_1x03_Pitch2.54mm
- U1: footprint IPC7351-Nominal:SOIC127P600X180-16 -> Housings_SOIC:SOIC-16_3.9x9.9mm_Pitch1.27mm
- U2: footprint Package_SO:MSOP-10_3x3mm_P0.5mm -> EtherkitKicadLibrary:MSOP-10
Connections:
- net +3V3: now also R15.2, R16.2
- net +4.3V: now also JP1.1 (A)
- net +5V: now also JP1.2 (B)
- net GND: now also J5.2
- net SCL: now also R15.1
- net SDA: now also R16.1
- net V_IN: now also J5.1
- net at J8.1 (Pin_1), U2.6 (CLK2): now also J19.1 (Pin_1); no longer P2.1 (In)
- net at C16.2, C17.1, R4.1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: now also T1.1 (AA); no longer T1.2 (AB)
- net at U3.2, U3.4: now also T1.5 (SB); no longer T1.3 (SA)
- net at U3.7, U3.9: now also T1.3 (SA); no longer T1.5 (SB)
- net at J6.1 (Pin_1), U1.9 (2A): now also T1.2 (AB); no longer T1.1 (AA)
- new net: J20.1 (Pin_1), P2.1 (In)
- no-connect marks 22 -> 23
Other:
- note removed: "Connect J15\nto J16 to \nremove\neffect of CC\nsmoother."
Changed lines of the file:
@@
 encoding utf-8
 Sheet 1 1
-Title "IQ_SDR Receiver"
-Date "2019-05-29"
+Title "Arduino HF SDR Receiver"
+Date "2019-07-11"
 Rev "0.1"
 Comp "Walla Walla University"
-Comment1 "Ultra Cheap HF QSD SDR"
-Comment2 ""
+Comment1 "Rob Frohne, KL7NA"
+Comment2 "Open Hardware License"
 Comment3 ""
 Comment4 ""
@@
 F 0 "U2" H 4100 1750 50  0000 C CNN
 F 1 "Si5351A-B-GT" H 3700 1300 50  0000 C CNN
-F 2 "Package_SO:MSOP-10_3x3mm_P0.5mm" H 4100 950 50  0001 C CNN
+F 2 "EtherkitKicadLibrary:MSOP-10" H 4100 950 50  0001 C CNN
 F 3 "https://www.silabs.com/documents/public/data-sheets/Si5351-B.pdf" H 3750 1650 50  0001 C CNN
 F 4 "X" H 4100 1750 50  0001 C CNN "Spice_Primitive"
@@
 P 9550 1950
 F 0 "A1" H 9550 1900 50  0000 C CNN
-F 1 "Arduino_Nano_v3.x" H 10050 1000 50  0000 C CNN
-F 2 "Module:Arduino_Nano" H 9700 1000 50  0001 L CNN
+F 1 "Arduino_Nano_v3.x" H 9650 650 50  0000 C CNN
+F 2 "Modules:Arduino_Nano" H 9700 1000 50  0001 L CNN
 F 3 "https://www.arduino.cc/en/uploads/Main/Arduino_Nano-Rev3.2-SCH.pdf" H 9550 950 50  0001 C CNN
 F 4 "R" H 9550 1950 50  0001 C CNN "Spice_Primitive"
@@
 F 0 "U1" V 2746 5970 50  0000 R CNN
 F 1 "FST3253" V 2655 5970 50  0000 R CNN
-F 2 "IPC7351-Nominal:SOIC127P600X180-16" H 2700 5900 50  0001 C CNN
+F 2 "Housings_SOIC:SOIC-16_3.9x9.9mm_Pitch1.27mm" H 2700 5900 50  0001 C CNN
 F 3 "https://www.onsemi.com/pub/Collateral/FST3253-D.pdf" H 2700 5700 50  0001 C CNN
 F 4 "DIST DIGIKEY FST3253MXFSCT-ND" H 2700 5800 60  0001 C CNN "BOM"
@@
 F 3 "~" H 5200 4450 50  0001 C CNN
 	1    5200 4450
-	1    0    0    -1
+	1    0    0    1
 $EndComp
 $Comp
@@
 Text Notes 7500 6700 0    50   ~ 0
 A very nice description of how op amp noise effects the noise figure\nis given in this data sheet \nhttps://www.ti.com/lit/ds/symlink/lmh6629.pdf \nin sections 7.3.4 and 7.3.5 (pages 24-7).   Finding an optimum R_g\n(input resistance for the inverting amplifier) seems to imply that\nthe optimum gets better as it goes to zero, assuming R_s is fixed.\nThe excess noise is approximately (e_n)^2+(i_n-)^2*(R_s+R_g)^2+4kTR_g, \nso minimizing e_n and i_n and R_g is\nthe best you can do.  The effect of i_n-  can be compared to e_n, by\nmultiplying by Rs_+Rg, so for R_g = 10 and R_s  = 50, e_n is more \nimportant in all the cases I've seen so far.  A nice calculator\nis at:\nhttp://dicks-website.eu/noisecalculator/index.html
-Text Notes 6600 3150 0    50   ~ 0
+Text Notes 5550 3300 0    50   ~ 0
 LT6231 has lower noise figure (4.7 dB), \nbut costs about 7 times as much\nas the SA5532.  LME49860 is \nintermediate option.  LM4562\ncould be even better (10.6 dB)\n2.7nV/sqrt(Hz).
 $Comp
@@
 $EndComp
 Wire Wire Line
-	4600 1950 4600 2400
-Connection ~ 4600 1950
-Wire Wire Line
 	4800 2550 4800 2650
 $Comp
@@
 $EndComp
 $Comp
-L power:GND #PWR09
+L power:GND #PWR08
 U 1 1 5CFDCC76
 P 1750 1750
-F 0 "#PWR09" H 1750 1500 50  0001 C CNN
+F 0 "#PWR08" H 1750 1500 50  0001 C CNN
 F 1 "GND" H 1755 1577 50  0000 C CNN
 F 2 "" H 1750 1750 50  0001 C CNN
@@
 $EndComp
 $Comp
-L power:GND #PWR010
+L power:GND #PWR09
 U 1 1 5D1D401E
 P 1750 4450
-F 0 "#PWR010" H 1750 4200 50  0001 C CNN
+F 0 "#PWR09" H 1750 4200 50  0001 C CNN
 F 1 "GND" H 1755 4277 50  0001 C CNN
 F 2 "" H 1750 4450 50  0001 C CNN
@@
 $EndComp
 $Comp
-L Jumper:Jumper_3_Bridged12 JP1
+L Jumper:Jumper_3_Bridged12 JP2
 U 1 1 5D208330
 P 8450 900
-F 0 "JP1" H 8450 1013 50  0000 C CNN
+F 0 "JP2" H 8450 1013 50  0000 C CNN
 F 1 "Jumper_3_Bridged12" H 8450 1013 50  0001 C CNN
-F 2 "" H 8450 900 50  0001 C CNN
+F 2 "Pin_Headers:Pin_Header_Straight_1x03_Pitch2.54mm" H 8450 900 50  0001 C CNN
 F 3 "~" H 8450 900 50  0001 C CNN
 	1    8450 900
@@
 F 0 "J3" H 1600 2700 50  0000 C CNN
 F 1 "V_IN pin header" H 1850 2600 50  0000 C CNN
-F 2 "" H 1450 2650 50  0001 C CNN
+F 2 "Pin_Headers:Pin_Header_Straight_1x02_Pitch2.54mm" H 1450 2650 50  0001 C CNN
 F 3 "~" H 1450 2650 50  0001 C CNN
 	1    1450 2650
@@
 $EndComp
 $Comp
-L power:GND #PWR08
+L power:GND #PWR010
 U 1 1 5D289723
-P 1650 2750
-F 0 "#PWR08" H 1650 2500 50  0001 C CNN
-F 1 "GND" H 1655 2577 50  0000 C CNN
-F 2 "" H 1650 2750 50  0001 C CNN
-F 3 "" H 1650 2750 50  0001 C CNN
-	1    1650 2750
+P 1800 2850
+F 0 "#PWR010" H 1800 2600 50  0001 C CNN
+F 1 "GND" H 1805 2677 50  0000 C CNN
+F 2 "" H 1800 2850 50  0001 C CNN
+F 3 "" H 1800 2850 50  0001 C CNN
+	1    1800 2850
 	1    0    0    -1
 $EndComp
@@
 	1    0    0    -1
 $EndComp
-$Comp
-L Connector_Generic:Conn_01x02 J5
-U 1 1 5D2A8ED8
-P 1850 2650
-F 0 "J5" H 1930 2642 50  0000 L CNN
-F 1 "Barrel Connector" H 1930 2551 50  0000 L CNN
-F 2 "" H 1850 2650 50  0001 C CNN
-F 3 "~" H 1850 2650 50  0001 C CNN
-	1    1850 2650
-	1    0    0    -1
-$EndComp
-Connection ~ 1650 2650
-Connection ~ 1650 2750
 Text Notes 650  2600 0    50   ~ 0
 V_IN is an optional\nDC Voltage for up to\n+30V.
@@
 Text Notes 650  3000 0    50   ~ 0
 Inputs for external\nDC input for op\namps.
-Connection ~ 8400 3850
-$Comp
-L power:PWR_FLAG #FLG0101
+$Comp
+L power:PWR_FLAG #FLG05
 U 1 1 5D47EB15
 P 8700 800
-F 0 "#FLG0101" H 8700 875 50  0001 C CNN
+F 0 "#FLG05" H 8700 875 50  0001 C CNN
 F 1 "PWR_FLAG" V 8700 928 50  0000 L CNN
 F 2 "" H 8700 800 50  0001 C CNN
@@
 	8700 800  8700 900
 $Comp
-L power:PWR_FLAG #FLG0102
+L power:PWR_FLAG #FLG04
 U 1 1 5D47F235
 P 8450 1150
-F 0 "#FLG0102" H 8450 1225 50  0001 C CNN
+F 0 "#FLG04" H 8450 1225 50  0001 C CNN
 F 1 "PWR_FLAG" V 8450 1277 50  0000 L CNN
 F 2 "" H 8450 1150 50  0001 C CNN
@@
 Wire Wire Line
 	8450 1150 8450 1250
-Text Notes 8350 1700 0    50   ~ 0
-Connect J15\nto J16 to \nremove\neffect of CC\nsmoother.
 Text Notes 6850 5200 0    50   ~ 0
 R9-10 can be\nup to 100\nwith LM4562.
 Text Notes 4700 4000 0    50   ~ 0
 Making T1 a step up\ntransformer makes\nthe S/N and NF better.
+$Comp
+L Jumper:Jumper_2_Open JP1
+U 1 1 5D205EC2
+P 7150 2100
+F 0 "JP1" V 7196 2012 50  0000 R CNN
+F 1 "smooth disable" V 7400 2400 50  0000 R CNN
+F 2 "Pin_Headers:Pin_Header_Straight_1x02_Pitch2.54mm" H 7150 2100 50  0001 C CNN
+F 3 "~" H 7150 2100 50  0001 C CNN
+	1    7150 2100
+	0    -1   -1   0
+$EndComp
+Wire Wire Line
+	7150 1900 7150 1800
+Wire Wire Line
+	7150 1800 7700 1800
+Connection ~ 7700 1800
+Wire Wire Line
+	7150 2300 7150 2550
+Wire Wire Line
+	7150 2550 8200 2550
+Connection ~ 8200 2550
+$Comp
+L Connector:Barrel_Jack_Switch J5
+U 1 1 5D263CFA
+P 2100 2750
+F 0 "J5" H 1870 2792 50  0000 R CNN
+F 1 "V_IN" H 1870 2701 50  0000 R CNN
+F 2 "Connectors:BARREL_JACK" H 2150 2710 50  0001 C CNN
+F 3 "https://www.cui.com/product/resource/pj-002a.pdf" H 2150 2710 50  0001 C CNN
+	1    2100 2750
+	-1   0    0    -1
+$EndComp
+Wire Wire Line
+	1650 2650 1800 2650
+Connection ~ 1650 2650
+Wire Wire Line
+	1800 2850 1650 2850
+Wire Wire Line
+	1650 2850 1650 2750
+Connection ~ 1800 2850
+NoConn ~ 1800 2750
+$Comp
+L Connector:Conn_01x01_Male J20
+U 1 1 5D381DCF
+P 4600 2200
+F 0 "J20" V 4708 2244 50  0000 L CNN
+F 1 "Conn_01x01_Male" V 4753 2244 50  0001 L CNN
+F 2 "Pin_Headers:Pin_Header_Straight_1x01_Pitch2.54mm" H 4600 2200 50  0001 C CNN
+F 3 "~" H 4600 2200 50  0001 C CNN
+	1    4600 2200
+	0    1    1    0
+$EndComp
+$Comp
+L Connector:Conn_01x01_Male J19
+U 1 1 5D383943
+P 4600 2150
+F 0 "J19" V 4708 2062 50  0000 R CNN
+F 1 "Conn_01x01_Male" V 4663 2062 50  0001 R CNN
+F 2 "Pin_Headers:Pin_Header_Straight_1x01_Pitch2.54mm" H 4600 2150 50  0001 C CNN
+F 3 "~" H 4600 2150 50  0001 C CNN
+	1    4600 2150
+	0    -1   -1   0
+$EndComp
+Connection ~ 4600 1950
+$Comp
+L Device:R R15
+U 1 1 5D5200C2
+P 10150 2950
+F 0 "R15" H 9950 3000 50  0000 L CNN
+F 1 "4.7k" H 9900 2900 50  0000 L CNN
+F 2 "Resistors_SMD:R_0805" V 10080 2950 50  0001 C CNN
+F 3 "~" H 10150 2950 50  0001 C CNN
+	1    10150 2950
+	1    0    0    -1
+$EndComp
+$Comp
+L Device:R R16
+U 1 1 5D520742
+P 10300 2950
+F 0 "R16" H 10350 2950 50  0000 L CNN
+F 1 "4.7k" H 10350 2850 50  0000 L CNN
+F 2 "Resistors_SMD:R_0805" V 10230 2950 50  0001 C CNN
+F 3 "~" H 10300 2950 50  0001 C CNN
+	1    10300 2950
+	1    0    0    -1
+$EndComp
+Wire Wire Line
+	10150 2800 10150 2450
+Wire Wire Line
+	10150 2450 10050 2450
+Wire Wire Line
+	10300 2800 10300 2350
+Wire Wire Line
+	10300 2350 10050 2350
+$Comp
+L power:+3.3V #PWR070
+U 1 1 5D5880C9
+P 9850 3100
+F 0 "#PWR070" H 9850 2950 50  0001 C CNN
+F 1 "+3.3V" H 9800 3250 50  0000 C CNN
+F 2 "" H 9850 3100 50  0001 C CNN
+F 3 "" H 9850 3100 50  0001 C CNN
+	1    9850 3100
+	1    0    0    -1
+$EndComp
+Wire Wire Line
+	9850 3100 10150 3100
+Wire Wire Line
+	10150 3100 10300 3100
+Connection ~ 10150 3100
 $EndSCHEMATC
