File: Receiver/IQ_SDR/IQ_SDR.sch (KiCad schematic (older format))
At the start: 97 parts, among them CON1 SJ1-3523N, J1 ANT, J10 LO_I, J11 LO_Q, J12 GNDA, J13 I_IN, J14 Q_IN, J15 +5V, J16 4.3V, J17 I_OUT, J18 Q_OUT, J19 Conn_01x01_Male, J2 GND, J20 Conn_01x01_Male, J3 V_IN pin header, J4 GND, J5 V_IN, J6 FIL_O, J7 CLK1, J8 CLK2, J9 CLK0, P1 BNC, P2 SMA, Q1 MMBT2222A-TP, T1 Transformer_1P_SS, U1 FST3253 or TS3A5017, U2 Si5351A-B-GT, U3 TS5A23157, U4 LM4562 or LT6231, U5 74ALVC74D, Y1 CX3225

Commit message: Added torroid data.
Parts:
- A1: symbol MCU_Module:Arduino_Nano_v3.x -> IQ_SDR-rescue:Arduino_Nano_v3.x-MCU_Module
- CON1: symbol dk_Barrel-Audio-Connectors:SJ1-3523N -> IQ_SDR-rescue:SJ1-3523N-dk_Barrel-Audio-Connectors
- L10, L4: Toroid (none) -> T37-6 13 turns
- Q1: symbol dk_Transistors-Bipolar-BJT-Single:MMBT2222A-TP -> IQ_SDR-rescue:MMBT2222A-TP-dk_Transistors-Bipolar-BJT-Single
- U5: symbol dk_Logic-Flip-Flops:SN74HC74N -> IQ_SDR-rescue:SN74HC74N-dk_Logic-Flip-Flops
- V1: symbol myspice:VSOURCE -> IQ_SDR-rescue:VSOURCE-myspice
Changed lines of the file:
@@
 EESchema Schematic File Version 4
-LIBS:IQ_SDR-cache
 EELAYER 30 0
 EELAYER END
@@
 $EndComp
 $Comp
-L MCU_Module:Arduino_Nano_v3.x A1
+L IQ_SDR-rescue:Arduino_Nano_v3.x-MCU_Module A1
 U 1 1 5D491311
 P 9550 1950
@@
 $EndComp
 $Comp
-L dk_Barrel-Audio-Connectors:SJ1-3523N CON1
+L IQ_SDR-rescue:SJ1-3523N-dk_Barrel-Audio-Connectors CON1
 U 1 1 5D491316
 P 10000 4050
@@
 Connection ~ 3000 1750
 $Comp
-L dk_Logic-Flip-Flops:SN74HC74N U5
+L IQ_SDR-rescue:SN74HC74N-dk_Logic-Flip-Flops U5
 U 1 1 5CF21139
 P 5800 1850
@@
 	1250 7250 1400 7250
 $Comp
-L myspice:VSOURCE V1
+L IQ_SDR-rescue:VSOURCE-myspice V1
 U 1 1 5D2E799E
 P 1050 6200
@@
 F 2 "Inductors_THT:L_Toroid_Vertical_L10.0mm_W5.0mm_P5.08mm" H 2100 4850 50  0001 C CNN
 F 3 "http://www.lodestonepacific.com/distrib/pdfs/Micrometals/RFA_Cat.pdf" H 2100 4850 50  0001 C CNN
+F 4 "T37-6 13 turns" H 2100 4850 50  0001 C CNN "Toroid"
 	1    2100 4850
 	1    0    0    -1
@@
 F 2 "Inductors_THT:L_Toroid_Vertical_L10.0mm_W5.0mm_P5.08mm" H 3500 4850 50  0001 C CNN
 F 3 "http://www.lodestonepacific.com/distrib/pdfs/Micrometals/RFA_Cat.pdf" H 3500 4850 50  0001 C CNN
+F 4 "T37-6 13 turns" H 3500 4850 50  0001 C CNN "Toroid"
 	1    3500 4850
 	1    0    0    -1
@@
 $EndComp
 $Comp
-L dk_Transistors-Bipolar-BJT-Single:MMBT2222A-TP Q1
+L IQ_SDR-rescue:MMBT2222A-TP-dk_Transistors-Bipolar-BJT-Single Q1
 U 1 1 5D24AC2F
 P 8100 2100

Commit message: Added in changes from the shop after failed merge.
Parts:
- C1, C10, C11, C12, C13, C14, C15, C16, C17, C18, C19, C2, C20, C21, C22, C23, C24, C25, C26, C27, C28, C29, C3, C30, C31, C32, C4, C5, C6, C7, C8, C9: symbol Device:C -> IQ_SDR-rescue:C-Device
- D1, D2: symbol Device:D_ALT -> IQ_SDR-rescue:D_ALT-Device
- J1, J10, J11, J12, J13, J14, J15, J16, J17, J18, J2, J4, J6, J7, J8, J9: symbol Connector_Generic:Conn_01x01 -> IQ_SDR-rescue:Conn_01x01-Connector_Generic
- J3: symbol Connector_Generic:Conn_01x02 -> IQ_SDR-rescue:Conn_01x02-Connector_Generic
- JP1: symbol Jumper:Jumper_2_Open -> IQ_SDR-rescue:Jumper_2_Open-Jumper
- JP2: symbol Jumper:Jumper_3_Bridged12 -> IQ_SDR-rescue:Jumper_3_Bridged12-Jumper
- L1, L10, L11, L12, L2, L3, L4, L5, L6, L7, L8, L9: symbol Device:L -> IQ_SDR-rescue:L-Device
- R1, R10, R11, R12, R13, R14, R15, R16, R2, R3, R4, R5, R6, R7, R8, R9: symbol Device:R -> IQ_SDR-rescue:R-Device
- T1: symbol Device:Transformer_1P_SS -> IQ_SDR-rescue:Transformer_1P_SS-Device
- U2: symbol Oscillator:Si5351A-B-GT -> IQ_SDR-rescue:Si5351A-B-GT-Oscillator
- U4: symbol Amplifier_Operational:NJM5532 -> IQ_SDR-rescue:NJM5532-Amplifier_Operational
Connections:
- net 1.5_GND: now reaches C16.2, C17.1, R4.1, R5.2, T1.1 (AA)
Other:
- note added: "Inductors in bandpass filters need to go to 1.5_GND, not GND.\nThey will short out the bias for the switches."
- note added: "Note: The switch numbers are not 0-3, but 1-4,\nso 00=>1, 01=>2, 10=>3, and 11=>4."
