File: Receiver/IQ_SDR/IQ_SDR.kicad_pcb (KiCad board)
At the start: 2 copper layers, 100 x 100 mm, 116 parts, among them CON1 SJ1-3523N, J1 ANT, J10 LO_I, J11 LO_Q, J12 GNDA, J13 I_IN, J14 Q_IN, J15 +5V, J16 4.3V, J17 I_OUT, J18 Q_OUT, J19 TX_I, J2 GND, J20 TX_O, J3 + V_IN -, J4 GND, J5 V_IN, J6 FIL_O, J7 CLK1, J8 CLK2, J9 CLK0, P1 BNC, P2 SMA, Q1 MMBT2222A-TP, T1 Transformer_1P_SS, U1 FST3253, U2 Si5351A, U3 TS5A23157, U4 LM4562 or LT6231, U5 74ALVC74D, Y1 CX3225

Commit message: Add inductor/transformer details.  Change U1 package type.  (Maybe should change the IC as we did in rev 0.1.)
Parts:
- C10: value 480pF -> 470pF
- C26, C27: value 0.002uF -> 2200pF
- C9: value 200pF -> 180pF
- J19: value TX_I -> Conn_01x01_Male
- J20: value TX_O -> Conn_01x01_Male
- J3: value + V_IN - -> V_IN pin header
- JP1: value 5->4.3V -> smooth disable
- JP2: value V_IN -> Jumper_3_Bridged12
- U1: footprint Housings_SOIC:SOIC-16_3.9x9.9mm_Pitch1.27mm -> Housings_SSOP:TSSOP-16_4.4x5mm_Pitch0.65mm
- U2: value Si5351A -> Si5351A-B-GT
Routing:
- net Net-(C6-Pad1): track 58.5 -> 67.6 mm
- net /B0: track 61.6 -> 55.5 mm
- net GND: track 658.2 -> 663.8 mm, vias 41 -> 46
- net Net-(J6-Pad1): track 22.1 -> 18.4 mm
- net Net-(C5-Pad1): track 73.7 -> 76.8 mm
- net +4.3V: track 135.8 -> 138.2 mm
- net Net-(C11-Pad1): track 66.0 -> 65.1 mm
- net Net-(C3-Pad2): track 6.05 -> 6.89 mm
- net Net-(C2-Pad1): track 49.1 -> 48.4 mm
- net Net-(C12-Pad1): track 56.0 -> 55.4 mm
