File: Transceiver/IQ_SDR/IQ_SDR.sch (KiCad schematic (older format))
At the start: 114 parts, among them CON1 SJ1-3523N, J1 GND, J10 GNDA, J11 I_IN, J12 Q_IN, J13 I_OUT, J14 Q_OUT, J2 FIL_I, J3 GND, J4 FIL_O, J5 CLK2, J6 CLK1, J7 CLK0, J8 LO_I, J9 LO_Q, P1 BNC, T1 Transformer_1P_SS, U1 FST3253, U2 Si5351A-B-GT, U3 TS5A23157, U4 FST3253, U5 SA5532 or LT6231, U6 74ALVC74D, Y1 CX3225

Commit message: Added PCB.
Parts:
- added R14, R15: 4.7k, Resistors_SMD:R_0805, symbol Device:R
- gave numbers to parts that had none: 1
- renumbered C5 to C1, C18 to C10, C23 to C11, C24 to C12, C25 to C13, C26 to C14, C27 to C15, C32 to C16, C33 to C17, C34 to C18, C35 to C19, C10 to C2, C37 to C20, C38 to C21, C39 to C22, C40 to C23, C41 to C24, C42 to C25, C43 to C26, C44 to C27, C46 to C28, C47 to C29, C11 to C3, C1 to C30, C2 to C31, C3 to C32, C4 to C33, C36 to C34, C6 to C35, C7 to C36, C8 to C37, C9 to C38, C45 to C39, C12 to C4, C19 to C40, C20 to C41, C21 to C42, C22 to C43, C48 to C44, C28 to C45, C29 to C46, C30 to C47, C31 to C48, C13 to C5, C14 to C6, C15 to C7, C16 to C8, C17 to C9, L5 to L1, L18 to L10, L19 to L11, L20 to L12, L1 to L13, L2 to L14, L3 to L15, L4 to L16, L9 to L17, L10 to L18, L11 to L19, L6 to L2, L12 to L20, L7 to L3, L8 to L4, L13 to L5, L14 to L6, L15 to L7, L16 to L8, L17 to L9, U5 to U4, U6 to U5, U4 to U6
Connections:
- wire segments 236 -> 240

Commit message: update in libraries for schematic
Parts:
- A1: symbol MCU_Module:Arduino_Nano_v3.x -> IQ_SDR-rescue:Arduino_Nano_v3.x-MCU_Module
Changed lines of the file:
@@
 EESchema Schematic File Version 4
-LIBS:IQ_SDR-cache
-EELAYER 29 0
+EELAYER 30 0
 EELAYER END
 $Descr USLedger 17000 11000
@@
 $EndComp
 $Comp
-L MCU_Module:Arduino_Nano_v3.x A1
+L IQ_SDR-rescue:Arduino_Nano_v3.x-MCU_Module A1
 U 1 1 5CEECC71
 P 11100 9000

Commit message: Moved the transceiver schematic from Reciever to Transceiver
Parts:
- removed C10, C13, C4: 390pF, Capacitors_SMD:C_0805, symbol Device:C
- removed C12, C3, C9: 680pF, Capacitors_SMD:C_0805, symbol Device:C
- removed C14, C5: 180pF, Capacitors_SMD:C_0805, symbol Device:C
- removed C15, C6: 100pF, Capacitors_SMD:C_0805, symbol Device:C
- removed C16, C17, C2, C22, C23, C25: 0.1uF, Capacitors_SMD:C_0805, symbol Device:C
- removed C28, C29: 10uF, Capacitors_SMD:C_0805, symbol Device:C
- removed C30, C31, C32, C35, C36, C37, C40, C45, C48, C7, C8: 1500pF, Capacitors_SMD:C_0805, symbol Device:C
- removed CON1: SJ1-3523N, digikey-footprints:Headphone_Jack_2.5mm_SJ1-3523N, symbol dk_Barrel-Audio-Connectors:SJ1-3523N
- removed D1: 1N914, Diodes_SMD:D_SOD-323, symbol Device:D_ALT
- removed J1, J3: GND, Connectors:PINTST, symbol Connector_Generic:Conn_01x01
- removed J11: I_IN, Connectors:PINTST, symbol Connector_Generic:Conn_01x01
- removed J12: Q_IN, Connectors:PINTST, symbol Connector_Generic:Conn_01x01
- removed J13: I_OUT, Connectors:PINTST, symbol Connector_Generic:Conn_01x01
- removed J14: Q_OUT, Connectors:PINTST, symbol Connector_Generic:Conn_01x01
- removed J4: FIL_O, Connectors:PINTST, symbol Connector_Generic:Conn_01x01
- removed L1, L15, L16, L19, L20, L23, L24, L9: 5.5uH, Inductors_THT:L_Toroid_Vertical_L10.0mm_W5.0mm_P5.08mm, symbol Device:L
- removed L10, L2: 2.0uH, Inductors_THT:L_Toroid_Vertical_L10.0mm_W5.0mm_P5.08mm, symbol Device:L
- removed L11, L3: 1.0uH, Inductors_THT:L_Toroid_Vertical_L10.0mm_W5.0mm_P5.08mm, symbol Device:L
- removed L4, L6: 0.46uH, Inductors_THT:L_Toroid_Vertical_L10.0mm_W5.0mm_P5.08mm, symbol Device:L
- removed L5: 2.6uH, Inductors_THT:L_Toroid_Vertical_L10.0mm_W5.0mm_P5.08mm, symbol Device:L
- removed L7: 0.27uH, Inductors_THT:L_Toroid_Vertical_L10.0mm_W5.0mm_P5.08mm, symbol Device:L
- removed L8: 0.13uH, Inductors_THT:L_Toroid_Vertical_L10.0mm_W5.0mm_P5.08mm, symbol Device:L
- removed Q1: BSD316SN, SMA:TUMT3, symbol dk_Transistors-FETs-MOSFETs-Single:2N7000
- removed R1, R6, R7: 2.2k, Resistors_SMD:R_0805, symbol Device:R
- removed R12: 100, Resistors_SMD:R_0805, symbol Device:R
- removed R14, R15: 4.7k, Resistors_SMD:R_0805, symbol Device:R
- removed R4, R5: 10k, Resistors_SMD:R_0805, symbol Device:R
- removed T1: Transformer_1P_SS, SMA:4_to_1_Transmission_Line_TransformerTHT, symbol Device:Transformer_1P_SS
- removed unit 1 of U4
- removed unit 3 of U4
- removed U6: FST3253, IPC7351-Nominal:SOIC127P600X180-16, symbol onsemi:FST3253
- removed V1: sin(0 10u {freq}), symbol myspice:VSOURCE
- added C10: 470pF, Capacitors_SMD:C_0805, symbol IQ_SDR-rescue:C-Device
- added C11, C5: 220pF, Capacitors_SMD:C_0805, symbol IQ_SDR-rescue:C-Device
- added C12, C6: 390pF, Capacitors_SMD:C_0805, symbol IQ_SDR-rescue:C-Device
- added C13, C2: 820pF, Capacitors_SMD:C_0805, symbol IQ_SDR-rescue:C-Device
- added C14, C4: 1.5nF, Capacitors_SMD:C_0805, symbol IQ_SDR-rescue:C-Device
- added C16, C25, C28, C3, C32, C40: 0.1uF, Capacitors_SMD:C_0805, symbol IQ_SDR-rescue:C-Device
- added C21, C22: 0.02uF, Capacitors_SMD:C_0805, symbol IQ_SDR-rescue:C-Device
- added C24, C29, C30, C36: 10uF, Capacitors_SMD:C_0805, symbol IQ_SDR-rescue:C-Device
- added C35: 1uF, Capacitors_SMD:C_0805, symbol IQ_SDR-rescue:C-Device
- added C37: 1u, Capacitors_SMD:C_0805, symbol IQ_SDR-rescue:C-Device
- added C44: 220pF, symbol Device:C
- added C50, C51, C52, C53, C54, C55, C56, C57, C58, C59, C60: 0.1uF, symbol Device:C
- added C61, C62: 470uF, symbol Device:CP1
- added C7: 47pF, Capacitors_SMD:C_0805, symbol IQ_SDR-rescue:C-Device
- added C8: 100pF, Capacitors_SMD:C_0805, symbol IQ_SDR-rescue:C-Device
- added C9: 180pF, Capacitors_SMD:C_0805, symbol IQ_SDR-rescue:C-Device
- added CON1: SJ1-3523N, digikey-footprints:Headphone_Jack_2.5mm_SJ1-3523N, symbol IQ_SDR-rescue:SJ1-3523N-dk_Barrel-Audio-Connectors
- added D1, D4, D5, D6, D7: 1N914, Diodes_SMD:D_SOD-323, symbol IQ_SDR-rescue:D_ALT-Device
- added D3: LED_Solid, symbol LED_Solid:LED_Solid
- added J13: I_IN, Connectors:PINTST, symbol IQ_SDR-rescue:Conn_01x01-Connector_Generic
- added J14: Q_IN, Connectors:PINTST, symbol IQ_SDR-rescue:Conn_01x01-Connector_Generic
- added J15: +5V, Connectors:PINTST, symbol IQ_SDR-rescue:Conn_01x01-Connector_Generic
- added J16: 4.3V, Connectors:PINTST, symbol IQ_SDR-rescue:Conn_01x01-Connector_Generic
- added J17: I_OUT, Connectors:PINTST, symbol IQ_SDR-rescue:Conn_01x01-Connector_Generic
- added J18: Q_OUT, Connectors:PINTST, symbol IQ_SDR-rescue:Conn_01x01-Connector_Generic
- added J19, J20: Conn_01x01_Male, Pin_Headers:Pin_Header_Straight_1x01_Pitch2.54mm, symbol Connector:Conn_01x01_Male
- added J2, J4: GND, Connectors:PINTST, symbol IQ_SDR-rescue:Conn_01x01-Connector_Generic
- added J21: V_CC, Connectors:PINTST, symbol IQ_SDR-rescue:Conn_01x01-Connector_Generic
- added J22: Ba, Connectors:PINTST, symbol IQ_SDR-rescue:Conn_01x01-Connector_Generic
- added J23: Bb, Connectors:PINTST, symbol IQ_SDR-rescue:Conn_01x01-Connector_Generic
- added J24: Cb, Connectors:PINTST, symbol IQ_SDR-rescue:Conn_01x01-Connector_Generic
- added J25: Ca, Connectors:PINTST, symbol IQ_SDR-rescue:Conn_01x01-Connector_Generic
- added J26: Gb, Connectors:PINTST, symbol IQ_SDR-rescue:Conn_01x01-Connector_Generic
- added J27: Ga, Connectors:PINTST, symbol IQ_SDR-rescue:Conn_01x01-Connector_Generic
- added J28, J29, J30, J31, J32, J33: Conn_01x02_Female, symbol Connector:Conn_01x02_Female
- added J3: V_IN pin header, Pin_Headers:Pin_Header_Straight_1x02_Pitch2.54mm, symbol IQ_SDR-rescue:Conn_01x02-Connector_Generic
- added J5: V_IN, Connectors:BARREL_JACK, symbol Connector:Barrel_Jack_Switch
- added J6: FIL_O, Connectors:PINTST, symbol IQ_SDR-rescue:Conn_01x01-Connector_Generic
- added J?: Conn_01x04_Male, symbol Connector:Conn_01x04_Male
- added JP1: smooth disable, Pin_Headers:Pin_Header_Straight_1x02_Pitch2.54mm, symbol IQ_SDR-rescue:Jumper_2_Open-Jumper
- added JP10, JP9: Jumper_NC_Small, symbol Device:Jumper_NC_Small
- added JP11, JP3, JP4, JP5, JP6, JP7, JP8: Jumper, symbol Device:Jumper
- added JP2: Jumper_3_Bridged12, Pin_Headers:Pin_Header_Straight_1x03_Pitch2.54mm, symbol IQ_SDR-rescue:Jumper_3_Bridged12-Jumper
- added L1: 1uH, Inductors_THT:L_Toroid_Vertical_L10.0mm_W5.0mm_P5.08mm, symbol IQ_SDR-rescue:L-Device
- added L10: 626nH, Inductors_THT:L_Toroid_Vertical_L10.0mm_W5.0mm_P5.08mm, symbol IQ_SDR-rescue:L-Device
- added L11: 1.7uH, Inductors_THT:L_Toroid_Vertical_L10.0mm_W5.0mm_P5.08mm, symbol IQ_SDR-rescue:L-Device
- added L15, L2: 2.4uH, Inductors_THT:L_Toroid_Vertical_L10.0mm_W5.0mm_P5.08mm, symbol IQ_SDR-rescue:L-Device
- added L25: 300uH, symbol Device:L
- added L3: 232nH, Inductors_THT:L_Toroid_Vertical_L10.0mm_W5.0mm_P5.08mm, symbol IQ_SDR-rescue:L-Device
- added L4: 497nH, Inductors_THT:L_Toroid_Vertical_L10.0mm_W5.0mm_P5.08mm, symbol IQ_SDR-rescue:L-Device
- added L5: 1.137uH, Inductors_THT:L_Toroid_Vertical_L10.0mm_W5.0mm_P5.08mm, symbol IQ_SDR-rescue:L-Device
- added L6: 1.98uH, Inductors_THT:L_Toroid_Vertical_L10.0mm_W5.0mm_P5.08mm, symbol IQ_SDR-rescue:L-Device
- added L7: 4uH, Inductors_THT:L_Toroid_Vertical_L10.0mm_W5.0mm_P5.08mm, symbol IQ_SDR-rescue:L-Device
- added L8: 7.2uH, Inductors_THT:L_Toroid_Vertical_L10.0mm_W5.0mm_P5.08mm, symbol IQ_SDR-rescue:L-Device
- added L9: 256nH, Inductors_THT:L_Toroid_Vertical_L10.0mm_W5.0mm_P5.08mm, symbol IQ_SDR-rescue:L-Device
- added P2, P3, P4: SMA, SMA:SMA_EDGE, symbol IQ_SDR-rescue:BNC-lt6231
- added Q1, Q10, Q11, Q6, Q7: MMBT2222A-TP, digikey-footprints:SOT-23-3, symbol IQ_SDR-rescue:MMBT2222A-TP-dk_Transistors-Bipolar-BJT-Single
- added Q2, Q3, Q4, Q5: 2N3904, Package_TO_SOT_THT:TO-92_Inline, symbol Transistor_BJT:2N3904
- added Q8, Q9: IRF510PBF, digikey-footprints:TO-220-3, symbol dk_Transistors-FETs-MOSFETs-Single:IRF510PBF
- added R1: 2.2k, Resistors_SMD:R_0805, symbol IQ_SDR-rescue:R-Device
- added R13: 100, Resistors_SMD:R_0805, symbol IQ_SDR-rescue:R-Device
- added R15, R16, R33, R34: 4.7k, Resistors_SMD:R_0805, symbol IQ_SDR-rescue:R-Device
- added R17, R18: 100, symbol Device:R
- added R19, R20, R23, R24: 22, symbol Device:R
- added R21, R22: 1k, symbol Device:R
- added R25: 2.2, symbol Device:R
- added R26, R27: 0, symbol Device:R
- added R28: 500, Resistors_SMD:R_0805, symbol IQ_SDR-rescue:R-Device
- added R29, R30: 47, symbol Device:R
- added R31, R32: 220, symbol Device:R
- added R35: 1.6k, Resistors_SMD:R_0805, symbol IQ_SDR-rescue:R-Device
- added R4: 10k, Resistors_SMD:R_0805, symbol IQ_SDR-rescue:R-Device
- added R5: 5.6k, Resistors_SMD:R_0805, symbol IQ_SDR-rescue:R-Device
- added R6: 2k, Resistors_SMD:R_0805, symbol IQ_SDR-rescue:R-Device
- added R7: 27k, Resistors_SMD:R_0805, symbol IQ_SDR-rescue:R-Device
- added R8: 1k, Resistors_SMD:R_0805, symbol IQ_SDR-rescue:R-Device
- added RLY1, RLY2: TX2SA-L-3V-Z, digikey-footprints:Relay_THT_EC2, symbol dk_Signal-Relays-Up-to-2-Amps:EC2-5NU
- added RV1, RV2: 10k, symbol Device:R_POT
- added T1: Transformer_1P_SS, IQ_SDR:Transformer_Toroid_Tapped_Secondary_Horizontal_D14.0mm_Amidon-T50, symbol IQ_SDR-rescue:Transformer_1P_SS-Device
- added T2, T3: Transformer_1P_1S, symbol Device:Transformer_1P_1S
- added T4: Transformer_SP_1S, symbol Device:Transformer_SP_1S
- added T5: BN43-6802, symbol Device:Transformer_1P_1S
- added unit 1 of U4
- added unit 3 of U4
- added U6: 1.6k, blue_pill:BLUEPILL, symbol blue_pill:BP
- A1: footprint Module:Arduino_Nano -> Modules:Arduino_Nano
- C1: symbol Device:C -> IQ_SDR-rescue:C-Device
- C15: renamed from C11; symbol Device:C -> IQ_SDR-rescue:C-Device
- C17: renamed from C18; symbol Device:C -> IQ_SDR-rescue:C-Device
- C18: renamed from C19; symbol Device:C -> IQ_SDR-rescue:C-Device
- C19: renamed from C20; symbol Device:C -> IQ_SDR-rescue:C-Device
- C20: renamed from C21; symbol Device:C -> IQ_SDR-rescue:C-Device
- C23: renamed from C24; symbol Device:C -> IQ_SDR-rescue:C-Device
- C26, C27: value 0.002uF -> 50pF; symbol Device:C -> IQ_SDR-rescue:C-Device
- C31: renamed from C44; value 0.1uF -> 10uF; symbol Device:C -> IQ_SDR-rescue:C-Device
- C33, C46: value 1500pF -> 160pF
- C34: value 0.01 -> 82pF
- C38, C42: value 1500pF -> 680pF
- C39: value 0.1uF -> 330pF
- C41: value 1500pF -> 220pF; footprint Capacitors_SMD:C_0805 -> (none)
- C43: value 1500pF -> 330pF
- C47: value 1500pF -> 82pF
- D2: symbol Device:D_ALT -> IQ_SDR-rescue:D_ALT-Device
- J1: renamed from J2; value FIL_I -> ANT; symbol Connector_Generic:Conn_01x01 -> IQ_SDR-rescue:Conn_01x01-Connector_Generic
- J10: renamed from J8; symbol Connector_Generic:Conn_01x01 -> IQ_SDR-rescue:Conn_01x01-Connector_Generic
- J11: renamed from J9; symbol Connector_Generic:Conn_01x01 -> IQ_SDR-rescue:Conn_01x01-Connector_Generic
- J12: renamed from J10; symbol Connector_Generic:Conn_01x01 -> IQ_SDR-rescue:Conn_01x01-Connector_Generic
- J7: renamed from J6; symbol Connector_Generic:Conn_01x01 -> IQ_SDR-rescue:Conn_01x01-Connector_Generic
- J8: renamed from J5; symbol Connector_Generic:Conn_01x01 -> IQ_SDR-rescue:Conn_01x01-Connector_Generic
- J9: renamed from J7; symbol Connector_Generic:Conn_01x01 -> IQ_SDR-rescue:Conn_01x01-Connector_Generic
- L12: value 0.46uH -> 300uH; footprint Inductors_THT:L_Toroid_Vertical_L10.0mm_W5.0mm_P5.08mm -> (none)
- L13, L21: value 5.5uH -> 1.18uH
- L14, L22: value 5.5uH -> 590nH
- L17: value 5.5uH -> 1.87uH
- L18: value 5.5uH -> 910nH
- P1: footprint (none) -> Connectors_TE-Connectivity:BNC_Socket_TYCO-AMP_LargePads
- R10: renamed from R9; value 10 -> 50; symbol Device:R -> IQ_SDR-rescue:R-Device
- R11: renamed from R10; value 4.7k -> 13k; symbol Device:R -> IQ_SDR-rescue:R-Device
- R12: renamed from R11; value 1.0k -> 13k; symbol Device:R -> IQ_SDR-rescue:R-Device
- R14: renamed from R13; symbol Device:R -> IQ_SDR-rescue:R-Device
- R2: symbol Device:R -> IQ_SDR-rescue:R-Device
- R3: value 10k -> 5.6k; symbol Device:R -> IQ_SDR-rescue:R-Device
- R9: renamed from R8; value 10 -> 50; symbol Device:R -> IQ_SDR-rescue:R-Device
- U1: value FST3253 -> FST3253 or TS3A5017; footprint IPC7351-Nominal:SOIC127P600X180-16 -> Housings_SSOP:TSSOP-16_4.4x5mm_Pitch0.65mm
- U2: footprint Package_SO:MSOP-10_3x3mm_P0.5mm -> EtherkitKicadLibrary:MSOP-10; symbol Oscillator:Si5351A-B-GT -> IQ_SDR-rescue:Si5351A-B-GT-Oscillator
- U4: value SA5532 or LT6231 -> LM4562 or LT6231; footprint SMA:DMP8 -> Housings_SOIC:SOIC-8_3.9x4.9mm_Pitch1.27mm; symbol Amplifier_Operational:NJM5532 -> IQ_SDR-rescue:NJM5532-Amplifier_Operational
- U5: symbol dk_Logic-Flip-Flops:SN74HC74N -> IQ_SDR-rescue:SN74HC74N-dk_Logic-Flip-Flops
- Y1: Frequency (none) -> 25MHz
Connections:
- net +3V3: now also C32.1, C40.1, D6.1 (K), D7.1 (K), R15.2, R16.2, RLY1.1 (COIL), RLY2.1 (COIL), U6.3V3 (3.3V); no longer C39.1
- net +5V: now also C36.1, J15.1 (Pin_1), J?.3 (Pin_3), JP1.2 (B), Q1.3 (C), R8.1, U6.5V; no longer C1.1, C18.1, C19.1, C34.1, R2.2, U1.16 (V+), U3.8 (V+)
- net B0: now also U6.PA4
- net B1: now also U6.PA5
- net GND: now also C11.2, C12.2, C13.2, C14.2, C2.2, C21.2, C22.2, C24.2, C25.1, C28.2, C32.2, C36.2, C37.2, C4.2, C40.2, C5.2, C52.2, C53.2, C56.2, C59.2, C6.2, C60.2, C61.2, C62.2, D1.1 (K), D3.1 (K), D5.1 (K), J2.1 (Pin_1), J4.1 (Pin_1), JP3.2, JP4.1, JP5.1, JP7.2, JP8.2, P2.2 (Ext), Q10.2 (E), Q11.2 (E), Q8.3 (S), Q9.3 (S), R17.2, R18.2, R19.2, R20.2, R23.2, R24.2, R28.2, R5.1, RV1.1, RV2.1, T2.3 (SA), T3.2 (AB), U4.4 (V-); no longer A1.29 (GND), A1.4 (GND), C41.2, P1.2 (Ext)
- net GNDA: now also C17.1, C16.2, C25.2, C37.1, L1.2, L10.2, L11.2, L15.2, L2.2, L3.2, L4.2, L9.2, P3.2 (Ext), Q6.2 (E), Q7.3 (C), R4.1, R5.2, T1.1 (AA), T1.4 (SC), U4.3 (+); no longer C23.2
- net MUTE: now also R1.2, U6.PA6
- net SCL: now also R15.1
- net SDA: now also R16.1
- net at J8.1 (Pin_1), U2.6 (CLK2): now also J19.1 (Pin_1)
- net at J7.1 (Pin_1), U2.9 (CLK1): now also T3.1 (AA)
- net at C26.1, R11.1: now also C29.2, J17.1 (Pin_1), J30.2 (Pin_2), J31.2 (Pin_2), U4.1
- net at C26.2, R11.2, R9.1: now also J28.2 (Pin_2), J30.1 (Pin_1), J31.1 (Pin_1), U4.2 (-)
- net at C27.2, R10.1, R12.2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: now also J29.2 (Pin_2), J32.1 (Pin_1), J33.1 (Pin_1)
- net at C27.1, R12.1, U4.7: now also C30.2, J18.1 (Pin_1), J32.2 (Pin_2), J33.2 (Pin_2)
- net at R14.1: now also CON1.3 (R)
- net at R2.1, R3.2, U1.7 (1A): now also C3.2
- net at U1.11 (2B2): now also C12.1, C8.1, L10.1
- net at U1.5 (1B2): now also C6.1, L4.1, L6.1
- net at R10.2, U3.10: now also C22.1, J14.1 (Pin_1), J29.1 (Pin_1)
- net at R9.2, U3.6: now also C21.1, J13.1 (Pin_1), J28.1 (Pin_1)
- net at U1.9 (2A): now also JP9.1
- net at U3.2, U3.4: now also R27.1
- net at U3.7, U3.9: now also R26.1
- net at R14.2: now also C30.1
- net at C47.1: now also L22.2, RLY1.10 (NC2)
- net at C46.1: now also L21.2, RLY1.8 (NO2); no longer L22.2
- net at L17.2, L21.1: now also C42.1
- net at L18.2, L22.1: now also C43.1; no longer C41.1
- net at U1.12 (2B3): now also C13.1, C9.1, L11.1
- net at U1.4 (1B3): now also C2.1, L1.1, L7.1
- net at U1.13 (2B4): now also C10.1, C14.1, L15.1
- net at U1.3 (1B4): now also C4.1, L2.1, L8.1
- net at L12.1: now also R31.1
- net V_CC: now reaches L12.2
- net V_CC: now also C19.1, C59.1, C60.1, C61.1, C62.1, J21.1 (Pin_1), JP2.2 (C), L25.2, Q6.3 (C), R25.1, R6.1, R7.1, U4.8 (V+)
- net at U1.10 (2B1): now also C11.1, C7.1, L9.1
- net at U1.6 (1B1): now also C5.1, L3.1, L5.1
- net at L13.1: now also C33.1, RLY1.5 (NO1)
- net at L14.1: now also C34.1, RLY1.3 (NC1)
- net at L14.2, L18.1: now also C39.1
- net at L13.2, L17.1: now also C38.1
- net at J1.1 (Pin_1): now also D2.1 (K), C3.1, D1.2 (A), JP6.2, R1.1, T2.4 (SB)
- net RF_IN: no longer names the net of P1.1 (In)
- net RF_IN: now also RLY2.9 (COM2); no longer D2.1 (K)
- new net: J20.1 (Pin_1), P2.1 (In)
- new net: C23.2, D3.2 (A), Q6.1 (B), R6.2
- new net: C10.2, L8.2
- new net: C9.2, L7.2
- new net: C24.1, Q1.1 (B), R8.2
- new net: C8.2, L6.2
- new net: C7.2, L5.2
- new net: J3.2 (Pin_2), J5.2, JP7.1
- new net: P1.2 (Ext), RLY2.4 (COM1)
- new net: CON1.1 (S), JP8.1
- new net: CON1.2 (T), R13.1
- new net: C29.1, R13.2
- new net: J6.1 (Pin_1), JP10.2, T1.2 (AB)
- new net: R26.2, T1.3 (SA)
- new net: R27.2, T1.5 (SB)
- new net: D4.2 (A), Q7.1 (B), R7.2
- new net: Q7.2 (E), R28.1
- new net: C54.1, C57.1, J26.1 (Pin_1), Q8.1 (G), R29.2
- new net: C54.2, T4.5 (S2)
- new net: D4.1 (K), D5.2 (A)
- new net: Q8.2 (D), T5.1 (AA)
- new net: C57.2, R31.2
- new net: J?.1 (Pin_1), U6.PA10
- new net: R35.1, U6.PA12
- new net: J?.2 (Pin_2), U6.PA9
- new net: C53.1, R29.1, RV1.2
- new net: D6.2 (A), Q10.3 (C), RLY1.12 (COIL)
- new net: JP11.1, P4.1 (In), RLY1.4 (COM1)
- new net: C35.2, RLY1.9 (COM2)
- new net: C55.1, C58.1, J27.1 (Pin_1), Q9.1 (G), R30.2
- new net: C55.2, T4.4 (S1)
- new net: Q9.2 (D), T5.2 (AB)
- new net: C58.2, R32.2
- new net: L25.1, R32.1
- new net: C56.1, R30.1, RV2.2
- new net: D7.2 (A), Q11.3 (C), RLY2.12 (COIL)
- new net: P4.2 (Ext), RLY2.5 (NO1), T5.3 (SA)
- new net: C35.1, RLY2.8 (NO2)
- new net: Q2.1 (E), R19.1
- new net: C41.2, C50.1, J22.1 (Pin_1), Q2.2 (B), Q4.2 (B), R17.1, R21.2
- new net: C41.1, J24.1 (Pin_1), Q2.3 (C), Q4.3 (C), R21.1, T4.1 (PR1)
- new net: Q4.1 (E), R23.1
- new net: C50.2, T3.4 (SB)
- new net: JP11.2, T5.4 (SB)
- new net: Q3.1 (E), R20.1
- new net: C44.2, C51.1, J23.1 (Pin_1), Q3.2 (B), Q5.2 (B), R18.1, R22.2
- new net: C44.1, J25.1 (Pin_1), Q3.3 (C), Q5.3 (C), R22.1, T4.3 (PR2)
- new net: Q5.1 (E), R24.1
- new net: C51.2, T3.3 (SA)
- new net: C52.1, R25.2, T4.2 (PM)
- new net: JP10.1, JP9.2, P3.1 (In)
- new net: Q10.1 (B), R33.2
- new net: Q11.1 (B), R34.2
- new net +4.3V: C1.1, C16.1, C18.1, C28.1, J16.1 (Pin_1), JP1.1 (A), JP2.1 (A), Q1.2 (E), R2.2, R4.2, RV1.3, RV2.3, U1.16 (V+), U3.8 (V+)
- new net ANT_RLY: R34.1, U6.PB9
- new net D_GND: A1.29 (GND), A1.4 (GND), J?.4 (Pin_4), JP3.1, R35.2, U6.G (GND)
- new net RX_ANT_+: JP6.1, RLY2.10 (NC2), RLY2.3 (NC1), T2.1 (AA)
- new net RX_ANT_-: JP4.2, JP5.2, T2.2 (AB)
- new net TX_BAND: R33.1, U6.PB8
- new net V_IN: J3.1 (Pin_1), J5.1, JP2.3 (B)
- no-connect marks 22 -> 51
Other:
- note added: "+5V"
- note added: "Antenna"
- note added: "BPF Responses:\n1.8MHz-4MHz\n4MHz-8MHz\n8MHz-16MHz\n16MHz-30MHZ"
- note added: "DGND"
- note added: "Emitter follower\nto smooth USB\n+5V."
- note added: "Experiment with ground\nloop problems\n"
- note added: "External DC in\nto run op amps\nand TX PA parts\nif desired."
- note added: "For ground loops"
- note added: "Inductors in bandpass filters need to go to 1.5_GND, not GND.\nThey will short out the bias for the switches."
- note added: "Inputs for external\nDC input for op\namps."
- note added: "Jumper\nand\nT2 for \nground \nloops.\nMay be\nunnecessary."
- note added: "LT6231 has lower noise figure (4.7 dB), \nbut costs about 7 times as much\nas the SA5532. LME49860 is \nintermediate option. LM4562\ncould be even better (10.6 dB)\n2.7nV/sqrt(Hz)."
- note added: "Making T1 a step up\ntransformer makes\nthe S/N and NF better."
- note added: "Note: The switch numbers are not 0-3, but 1-4,\nso 00=>1, 01=>2, 10=>3, and 11=>4."
- note added: "Optional"
- note added: "Oscillator\nOut"
- note added: "Populate the Blue Pill or the Nano,\nbut not both."
- note added: "R9-10 can be\nup to 100\nwith LM4562."
- note added: "RX"
- note added: "Serial programming\nheader"
- note added: "TX"
- note added: "To fix the blue pill\npull up value problem\n"
- note added: "V_IN is an optional\nDC Voltage for up to\n+30V."
- note added: "Voltage Reference\nfor Mixers and \nOp Amps\n"
- note added: "We could use differential amplifiers. \n(Switch the mixer\nchips around.) For a second order\nMFB op amp design see this, making\nit differential. \nhttps://webench.ti.com/filter-design-tool/export/11"
- note removed: ".param freq=10000000"
- note removed: ".param if_freq={freq + 1000}"
- note removed: "LT6231 has lower noise figure (6 dB), \nbut costs about 7 times as much\nas the SA5532."
- moved on the sheet: C1, C15, C17, C18, C19, C20, C23, C26, C27, C31, D2, J1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
